Commit message: IK 수정, Rviz 연결

File: src/open_manipulator_description/urdf/omx/omx_arm.urdf.xacro (robot description, xacro)
@@ -96,5 +96,5 @@
       <parent link="${prefix}link3"/>
       <child link="${prefix}link4"/>
-      <origin xyz="0.024 0 0.128" rpy="0 0 0"/>
+      <origin xyz="0.024 0 0.128" rpy="0 -1.5708 0"/>
       <axis xyz="0 1 0"/>
       <limit velocity="4.8" effort="1000" lower="${-1.5}" upper="${1.4}" />
